File: connectors.kicad_sch (KiCad schematic)
At the start: 26 parts, among them IC4 LDL1117S33R, J10 Conn_01x02_Pin, J2 Conn_01x04_Pin, J3 USB_C_Receptacle_USB2.0_16P, J4 Conn_01x02_Pin, J5 Conn_01x03_Pin, J6 Conn_01x03_Pin, J7 Conn_01x03_Pin, J8 Conn_01x03_Pin, J9 Conn_01x03_Pin, Q1 PMOS, Q2 PMOS, U3 CP2102N-Axx-xQFN20

Commit message: I2C change to SPI, add USART1
Changed lines of the file:
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@@
+		)
+	)
+	(hierarchical_label "USART2_TX"
+		(shape input)
+		(at 256.54 39.37 0)
+		(effects
+			(font
+				(size 1.27 1.27)
+			)
+			(justify left)
+		)
+	)
+	(hierarchical_label "USART2_RX"
+		(shape input)
+		(at 256.54 35.56 0)
+		(effects
+			(font
+				(size 1.27 1.27)
+			)
+			(justify left)
 		)
 	)

Commit message: I2C change to SPI, add USART1
Parts:
- added J11: Conn_01x03_Pin, symbol Connector:Conn_01x03_Pin
Connections:
- net GND: now also J11.3 (Pin_3)
- net USART2_RX: now also J11.2 (Pin_2)
- net USART2_TX: now also J11.1 (Pin_1)
Other:
- note added: "Camera connector"
- moved on the sheet: J10

Commit message: TCXO
Parts:
- C28: renamed from C21; footprint (none) -> Capacitor_SMD:C_0603_1608Metric_Pad1.08x0.95mm_HandSolder
- C29: renamed from C15; footprint (none) -> Capacitor_SMD:C_0603_1608Metric_Pad1.08x0.95mm_HandSolder
- C30: renamed from C9; footprint (none) -> Capacitor_SMD:C_0603_1608Metric_Pad1.08x0.95mm_HandSolder
- C31: renamed from C11; footprint (none) -> Capacitor_SMD:C_0603_1608Metric_Pad1.08x0.95mm_HandSolder
- C32: renamed from C12; footprint (none) -> Capacitor_SMD:C_0603_1608Metric_Pad1.08x0.95mm_HandSolder
- C33: renamed from C10; footprint (none) -> Capacitor_SMD:C_0603_1608Metric_Pad1.08x0.95mm_HandSolder
- C34: renamed from C22; footprint (none) -> Capacitor_SMD:C_0603_1608Metric_Pad1.08x0.95mm_HandSolder
- IC4: footprint SOT230P700X180-4N -> (none)
- Q1: footprint (none) -> Inductor_SMD:L_0402_1005Metric_Pad0.77x0.64mm_HandSolder
- R4: renamed from R12; footprint (none) -> Resistor_SMD:R_0603_1608Metric_Pad0.98x0.95mm_HandSolder
- R5: renamed from R13; footprint (none) -> Resistor_SMD:R_0603_1608Metric_Pad0.98x0.95mm_HandSolder
- R6: renamed from R10; footprint (none) -> Resistor_SMD:R_0603_1608Metric_Pad0.98x0.95mm_HandSolder
- R7: renamed from R11; footprint (none) -> Resistor_SMD:R_0603_1608Metric_Pad0.98x0.95mm_HandSolder
- R8: renamed from R9; footprint (none) -> Resistor_SMD:R_0603_1608Metric_Pad0.98x0.95mm_HandSolder
- renumbered J8 to J10, J4 to J2, J2 to J4, J10 to J5, J5 to J6, J9 to J8, J6 to J9, U3 to U4
