File: flight_controller.kicad_sch (KiCad schematic)
At the start: 31 parts, among them IC1 MAX-F10S-00B, J1 Conn_Coaxial, U1 STM32WL55CCUx, U4 AT25xxx, Y1 Crystal

Commit message: I2C change to SPI, add USART1
Connections:
- net Sensor/I2C1_SCL is gone; now on net SPI2_SCK: U1.17 (PA9)
- net Sensor/I2C1_SDA is gone; now on net SPI2_MOSI: U1.33 (PA10)
- net Sensor/I2C2_SCL is gone; now on net I2C2_SCL: U1.35 (PA12)
- net Sensor/I2C2_SDA is gone; now on net I2C2_SDA: U1.34 (PA11)
- net Sensor/LSM6_INT1 is gone; now on net F10S_RESET: U1.32 (PB12)
- net Connectors/SERWO3_PWM: now also U1.15 (PA7); no longer U1.9 (PA2)
- net Connectors/SERWO4_PWM: now also U1.16 (PA8); no longer U1.10 (PA3)
- net F10S_RESET: no longer U1.12 (PA4)
- net Sensor/BMP581_INT: now also U1.14 (PA6); no longer U1.16 (PA8)
- net SPI2_CS: now reaches U1.31 (PB2)
- net SPI2_CS: now also U4.1 (~{CS})
- net LSM6_INT1: now reaches U1.38 (PC13)
- net LSM6_INT2: now reaches U1.39 (PC14)
- net IIS2_RDY: now reaches U1.40 (PC15)
- net Sensor/SPI1_CS3: now reaches U1.43 (PA15)
- net I2C3_SCL renamed I2C2_SCL
- net I2C2_SCL: no longer U1.15 (PA7)
- net I2C3_SDA renamed I2C2_SDA
- net I2C2_SDA: no longer U1.2 (PB4)
- net SPI1_CLK renamed SPI2_SCK
- net SPI2_SCK: no longer U1.1 (PB3)
- net SPI1_CS renamed SPI2_MISO
- net SPI2_MISO: now also U4.2 (MISO); no longer U4.1 (~{CS})
- removed net SPI1_MISO: U1.14 (PA6), U4.2 (MISO)
- net SPI1_MOSI renamed SPI2_MOSI
- net SPI2_MOSI: no longer U1.3 (PB5)
- new net Connectors/USART2_RX: U1.9 (PA2)
- new net Connectors/USART2_TX: U1.10 (PA3)
- new net Sensor/SPI1_CS1: U1.2 (PB4)
- new net Sensor/SPI1_CS2: U1.12 (PA4)
- new net Sensor/SPI1_MOSI: U1.3 (PB5)
- new net Sensor/SPI1_SCK: U1.1 (PB3)
- no-connect marks 20 -> 15
Other:
- sheet Connectors ports: added USART2_RX, USART2_TX; removed none
- sheet Sensor ports: added IIS2_RDY, LSM6_INT2, SPI1_CS1, SPI1_CS2, SPI1_CS3, SPI1_MOSI, SPI1_SCK; removed I2C1_SCL, I2C1_SDA, I2C2_SCL, I2C2_SDA
- moved on the sheet: C1, C10, C13, C14, C2, C3, C4, C5, C9, J1, L1, L2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

Commit message: TCXO
Parts:
- removed Y1: Crystal, symbol Device:Crystal
- added Y1: FT3MNTUM-32.0-T1, Crystal:Crystal_SMD_Abracon_ABM8AIG-4Pin_3.2x2.5mm, symbol Device:Crystal_GND23
- C1: renamed from C28; footprint (none) -> Capacitor_SMD:C_0402_1005Metric_Pad0.74x0.62mm_HandSolder
- C10: footprint (none) -> Capacitor_SMD:C_0402_1005Metric_Pad0.74x0.62mm_HandSolder
- C11: renamed from C9; footprint (none) -> Capacitor_SMD:C_0402_1005Metric_Pad0.74x0.62mm_HandSolder
- C12: renamed from C20; footprint (none) -> Capacitor_SMD:C_0603_1608Metric_Pad1.08x0.95mm_HandSolder
- C13: renamed from C19; footprint (none) -> Capacitor_SMD:C_0603_1608Metric_Pad1.08x0.95mm_HandSolder
- C14: renamed from C29; footprint (none) -> Capacitor_SMD:C_0603_1608Metric_Pad1.08x0.95mm_HandSolder
- C15: renamed from C23; footprint (none) -> Capacitor_SMD:C_0603_1608Metric_Pad1.08x0.95mm_HandSolder
- C16: renamed from C24; footprint (none) -> Capacitor_SMD:C_0603_1608Metric_Pad1.08x0.95mm_HandSolder
- C17: renamed from C25; footprint (none) -> Capacitor_SMD:C_0603_1608Metric_Pad1.08x0.95mm_HandSolder
- C18: renamed from C26; footprint (none) -> Capacitor_SMD:C_0603_1608Metric_Pad1.08x0.95mm_HandSolder
- C19: renamed from C27; footprint (none) -> Capacitor_SMD:C_0603_1608Metric_Pad1.08x0.95mm_HandSolder
- C2: renamed from C14; value 18p -> 10p; footprint (none) -> Capacitor_SMD:C_0603_1608Metric_Pad1.08x0.95mm_HandSolder
- C3: renamed from C13; value 18p -> 10p; footprint (none) -> Capacitor_SMD:C_0603_1608Metric_Pad1.08x0.95mm_HandSolder
- C4: renamed from C5; footprint (none) -> Capacitor_SMD:C_0402_1005Metric_Pad0.74x0.62mm_HandSolder
- C5, C6: renamed from C4; footprint (none) -> Capacitor_SMD:C_0402_1005Metric_Pad0.74x0.62mm_HandSolder
- C7: renamed from C3; footprint (none) -> Capacitor_SMD:C_0402_1005Metric_Pad0.74x0.62mm_HandSolder
- C8: renamed from C2; footprint (none) -> Capacitor_SMD:C_0402_1005Metric_Pad0.74x0.62mm_HandSolder
- C9: renamed from C1; footprint (none) -> Capacitor_SMD:C_0402_1005Metric_Pad0.74x0.62mm_HandSolder
- IC1: footprint MAXF10S00B -> (none)
- L1: footprint (none) -> Inductor_SMD:L_0402_1005Metric_Pad0.77x0.64mm_HandSolder
- L2: renamed from L3; footprint (none) -> Inductor_SMD:L_0402_1005Metric_Pad0.77x0.64mm_HandSolder
- L3: renamed from L2; footprint (none) -> Inductor_SMD:L_0402_1005Metric_Pad0.77x0.64mm_HandSolder
- L4: renamed from L6; footprint (none) -> Inductor_SMD:L_0402_1005Metric_Pad0.77x0.64mm_HandSolder
- L5: renamed from L1; footprint (none) -> Inductor_SMD:L_0402_1005Metric_Pad0.77x0.64mm_HandSolder
- R1: renamed from R14; footprint (none) -> Resistor_SMD:R_0603_1608Metric_Pad0.98x0.95mm_HandSolder
- renumbered U4 to U1, U1 to U2
Connections:
- net GND: now also Y1.1 (G), Y1.2 (G)
- net OSC_IN: now also Y1.4 (1)
- net OSC_OUT: now also Y1.3 (4)
