File: sensor.kicad_sch (KiCad schematic)
At the start: 19 parts, among them IC2 LSM6DSV80XTR, IC3 IIS2MDCTR, U2 BMP581

Commit message: I2C change to SPI, add USART1
Parts:
- removed R3, R4, R5, R6, R7, R8: 10k, symbol Device:R_Small
Connections:
- net I2C2_SCL is gone; now on net SPI1_SCK: U2.2 (SCK)
- net I2C2_SDA is gone; now on net SPI1_MOSI: U2.4 (SDI)
- net +3.3V: no longer IC2.1 (SDO/SA0), IC2.12 (CS), IC3.3 (CS)
- net GND: now also IC2.2 (SDX), IC2.3 (SCX), IC3.2 (NC_1); no longer U2.5 (SDO)
- net I2C1_SCL renamed SPI1_SCK
- net SPI1_SCK: now also IC3.1 (SCL/SPC)
- net I2C1_SDA renamed SPI1_MOSI
- net SPI1_MOSI: now also IC3.4 (SDA/SDI/SDO)
- removed net I2C_SCL: IC2.3 (SCX), IC3.1 (SCL/SPC)
- removed net I2C_SDA: IC2.2 (SDX), IC3.4 (SDA/SDI/SDO)
- net LSM6_DRDY renamed IIS2_RDY
- net IIS2_RDY: no longer IC2.9 (INT2)
- net VDDIO: no longer names the net of R2.2, U2.1 (VDDIO)
- net VDDIO: no longer U2.6 (CSB)
- new net LSM6_INT2: IC2.9 (INT2)
- new net SPI1_CS1: IC2.12 (CS)
- new net SPI1_CS2: IC3.3 (CS)
- new net SPI1_CS3: U2.6 (CSB)
- no-connect marks 5 -> 6

Commit message: TCXO
Parts:
- C20: renamed from C8; footprint (none) -> Capacitor_SMD:C_0603_1608Metric_Pad1.08x0.95mm_HandSolder
- C21: renamed from C3; footprint (none) -> Capacitor_SMD:C_0603_1608Metric_Pad1.08x0.95mm_HandSolder
- C22: renamed from C4; footprint (none) -> Capacitor_SMD:C_0603_1608Metric_Pad1.08x0.95mm_HandSolder
- C23: renamed from C7; footprint (none) -> Capacitor_SMD:C_0603_1608Metric_Pad1.08x0.95mm_HandSolder
- C24: renamed from C6; footprint (none) -> Capacitor_SMD:C_0603_1608Metric_Pad1.08x0.95mm_HandSolder
- C25: renamed from C5; footprint (none) -> Capacitor_SMD:C_0603_1608Metric_Pad1.08x0.95mm_HandSolder
- C26: renamed from C1; footprint (none) -> Capacitor_SMD:C_0603_1608Metric_Pad1.08x0.95mm_HandSolder
- C27: renamed from C2; footprint (none) -> Capacitor_SMD:C_0603_1608Metric_Pad1.08x0.95mm_HandSolder
- IC2: renamed from IC3; footprint IIS2MDCTR -> (none)
- IC3: renamed from IC2; footprint LSM6DSV16BXTR -> (none)
- R2: footprint (none) -> Resistor_SMD:R_0603_1608Metric_Pad0.98x0.95mm_HandSolder
- R3: renamed from R1; footprint (none) -> Resistor_SMD:R_0603_1608Metric_Pad0.98x0.95mm_HandSolder
- U3: renamed from U2; footprint BMP581 -> (none)
Changed lines of the file:
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@@
 		(dnp no)
 		(fields_autoplaced yes)
-		(property "Reference" "C3"
+		(property "Reference" "C21"
 			(at 66.04 90.1762 0)
 			(show_name no)
@@
 			)
 		)
-		(property "Footprint" ""
+		(property "Footprint" "Capacitor_SMD:C_0603_1608Metric_Pad1.08x0.95mm_HandSolder"
 			(at 63.5 91.44 0)
 			(hide yes)
@@
 			(project "flight_controller"
 				(path "/6af40c3f-be19-463b-a9b6-2f3cba853d02/0704ef58-62bc-45a1-abb2-7b7b5f193951"
-					(reference "C3")
+					(reference "C21")
 					(unit 1)
 				)
@@
 		(dnp no)
 		(fields_autoplaced yes)
-		(property "Reference" "IC2"
+		(property "Reference" "IC3"
 			(at 87.2333 45.72 0)
 			(show_name no)
@@
 			)
 		)
-		(property "Footprint" "LSM6DSV16BXTR"
+		(property "Footprint" ""
 			(at 96.52 148.26 0)
 			(hide yes)
@@
 			(project "flight_controller"
 				(path "/6af40c3f-be19-463b-a9b6-2f3cba853d02/0704ef58-62bc-45a1-abb2-7b7b5f193951"
-					(reference "IC2")
+					(reference "IC3")
 					(unit 1)
 				)
@@
 		(dnp no)
 		(fields_autoplaced yes)
-		(property "Reference" "IC3"
+		(property "Reference" "IC2"
 			(at 83.82 143.51 0)
 			(show_name no)
@@
 			)
 		)
-		(property "Footprint" "IIS2MDCTR"
+		(property "Footprint" ""
 			(at 101.6 246.05 0)
 			(hide yes)
@@
 			(project "flight_controller"
 				(path "/6af40c3f-be19-463b-a9b6-2f3cba853d02/0704ef58-62bc-45a1-abb2-7b7b5f193951"
-					(reference "IC3")
+					(reference "IC2")
 					(unit 1)
 				)
@@
 		(dnp no)
 		(fields_autoplaced yes)
-		(property "Reference" "#PWR09"
+		(property "Reference" "#PWR021"
 			(at 110.49 179.07 0)
 			(hide yes)
@@
 			(project "flight_controller"
 				(path "/6af40c3f-be19-463b-a9b6-2f3cba853d02/0704ef58-62bc-45a1-abb2-7b7b5f193951"
-					(reference "#PWR09")
+					(reference "#PWR021")
 					(unit 1)
 				)
@@
 		(dnp no)
 		(fields_autoplaced yes)
-		(property "Reference" "C7"
+		(property "Reference" "C23"
 			(at 118.11 161.2962 0)
 			(show_name no)
@@
 			)
 		)
-		(property "Footprint" ""
+		(property "Footprint" "Capacitor_SMD:C_0603_1608Metric_Pad1.08x0.95mm_HandSolder"
 			(at 115.57 162.56 0)
 			(hide yes)
@@
 			(project "flight_controller"
 				(path "/6af40c3f-be19-463b-a9b6-2f3cba853d02/0704ef58-62bc-45a1-abb2-7b7b5f193951"
-					(reference "C7")
+					(reference "C23")
 					(unit 1)
 				)
@@
 		(dnp no)
 		(fields_autoplaced yes)
-		(property "Reference" "#PWR012"
+		(property "Reference" "#PWR025"
 			(at 245.11 85.09 0)
 			(hide yes)
@@
 			(project "flight_controller"
 				(path "/6af40c3f-be19-463b-a9b6-2f3cba853d02/0704ef58-62bc-45a1-abb2-7b7b5f193951"
-					(reference "#PWR012")
+					(reference "#PWR025")
 					(unit 1)
 				)
@@
 		(dnp no)
 		(fields_autoplaced yes)
-		(property "Reference" "C6"
+		(property "Reference" "C24"
 			(at 127 161.2962 0)
 			(show_name no)
@@
 			)
 		)
-		(property "Footprint" ""
+		(property "Footprint" "Capacitor_SMD:C_0603_1608Metric_Pad1.08x0.95mm_HandSolder"
 			(at 124.46 162.56 0)
 			(hide yes)
@@
 			(project "flight_controller"
 				(path "/6af40c3f-be19-463b-a9b6-2f3cba853d02/0704ef58-62bc-45a1-abb2-7b7b5f193951"
-					(reference "C6")
+					(reference "C24")
 					(unit 1)
 				)
@@
 		(dnp no)
 		(fields_autoplaced yes)
-		(property "Reference" "#PWR01"
+		(property "Reference" "#PWR023"
 			(at 227.33 69.85 0)
 			(hide yes)
@@
 			(project "flight_controller"
 				(path "/6af40c3f-be19-463b-a9b6-2f3cba853d02/0704ef58-62bc-45a1-abb2-7b7b5f193951"
-					(reference "#PWR01")
+					(reference "#PWR023")
 					(unit 1)
 				)
@@
 		(dnp no)
 		(fields_autoplaced yes)
-		(property "Reference" "C8"
+		(property "Reference" "C20"
 			(at 54.61 165.1062 0)
 			(show_name no)
@@
 			)
 		)
-		(property "Footprint" ""
+		(property "Footprint" "Capacitor_SMD:C_0603_1608Metric_Pad1.08x0.95mm_HandSolder"
 			(at 52.07 166.37 0)
 			(hide yes)
@@
 			(project "flight_controller"
 				(path "/6af40c3f-be19-463b-a9b6-2f3cba853d02/0704ef58-62bc-45a1-abb2-7b7b5f193951"
-					(reference "C8")
+					(reference "C20")
 					(unit 1)
 				)
@@
 		(dnp no)
 		(fields_autoplaced yes)
-		(property "Reference" "U2"
+		(property "Reference" "U3"
 			(at 245.11 90.0998 0)
 			(show_name no)
@@
 			)
 		)
-		(property "Footprint" "BMP581"
+		(property "Footprint" ""
 			(at 241.3 181.28 0)
 			(hide yes)
@@
 			(project "flight_controller"
 				(path "/6af40c3f-be19-463b-a9b6-2f3cba853d02/0704ef58-62bc-45a1-abb2-7b7b5f193951"
-					(reference "U2")
+					(reference "U3")
 					(unit 1)
 				)
@@
 		(dnp no)
 		(fields_autoplaced yes)
-		(property "Reference" "#PWR04"
+		(property "Reference" "#PWR022"
 			(at 200.66 83.82 0)
 			(hide yes)
@@
 			(project "flight_controller"
 				(path "/6af40c3f-be19-463b-a9b6-2f3cba853d02/0704ef58-62bc-45a1-abb2-7b7b5f193951"
-					(reference "#PWR04")
+					(reference "#PWR022")
 					(unit 1)
 				)
@@
 		(dnp no)
 		(fields_autoplaced yes)
-		(property "Reference" "#PWR08"
+		(property "Reference" "#PWR015"
 			(at 60.96 179.07 0)
 			(hide yes)
@@
 			(project "flight_controller"
 				(path "/6af40c3f-be19-463b-a9b6-2f3cba853d02/0704ef58-62bc-45a1-abb2-7b7b5f193951"
-					(reference "#PWR08")
+					(reference "#PWR015")
 					(unit 1)
 				)
@@
 		(dnp no)
 		(fields_autoplaced yes)
-		(property "Reference" "#PWR010"
+		(property "Reference" "#PWR020"
 			(at 107.95 147.32 0)
 			(hide yes)
@@
 			(project "flight_controller"
 				(path "/6af40c3f-be19-463b-a9b6-2f3cba853d02/0704ef58-62bc-45a1-abb2-7b7b5f193951"
-					(reference "#PWR010")
+					(reference "#PWR020")
 					(unit 1)
 				)
@@
 		(dnp no)
 		(fields_autoplaced yes)
-		(property "Reference" "#PWR040"
+		(property "Reference" "#PWR016"
 			(at 62.23 77.47 0)
 			(hide yes)
@@
 			(project "flight_controller"
 				(path "/6af40c3f-be19-463b-a9b6-2f3cba853d02/0704ef58-62bc-45a1-abb2-7b7b5f193951"
-					(reference "#PWR040")
+					(reference "#PWR016")
 					(unit 1)
 				)
@@
 		(dnp no)
 		(fields_autoplaced yes)
-		(property "Reference" "R1"
+		(property "Reference" "R3"
 			(at 229.87 72.3899 0)
 			(show_name no)
@@
 			)
 		)
-		(property "Footprint" ""
+		(property "Footprint" "Resistor_SMD:R_0603_1608Metric_Pad0.98x0.95mm_HandSolder"
 			(at 227.33 73.66 0)
 			(hide yes)
@@
 			(project "flight_controller"
 				(path "/6af40c3f-be19-463b-a9b6-2f3cba853d02/0704ef58-62bc-45a1-abb2-7b7b5f193951"
-					(reference "R1")
+					(reference "R3")
 					(unit 1)
 				)
@@
 		(dnp no)
 		(fields_autoplaced yes)
-		(property "Reference" "#PWR06"
+		(property "Reference" "#PWR019"
 			(at 105.41 62.23 0)
 			(hide yes)
@@
 			(project "flight_controller"
 				(path "/6af40c3f-be19-463b-a9b6-2f3cba853d02/0704ef58-62bc-45a1-abb2-7b7b5f193951"
-					(reference "#PWR06")
+					(reference "#PWR019")
 					(unit 1)
 				)
@@
 		(dnp no)
 		(fields_autoplaced yes)
-		(property "Reference" "C4"
+		(property "Reference" "C22"
 			(at 107.95 73.6662 0)
 			(show_name no)
@@
 			)
 		)
-		(property "Footprint" ""
+		(property "Footprint" "Capacitor_SMD:C_0603_1608Metric_Pad1.08x0.95mm_HandSolder"
 			(at 105.41 74.93 0)
 			(hide yes)
@@
 			(project "flight_controller"
 				(path "/6af40c3f-be19-463b-a9b6-2f3cba853d02/0704ef58-62bc-45a1-abb2-7b7b5f193951"
-					(reference "C4")
+					(reference "C22")
 					(unit 1)
 				)
@@
 		(dnp no)
 		(fields_autoplaced yes)
-		(property "Reference" "C1"
+		(property "Reference" "C26"
 			(at 203.2 72.3962 0)
 			(show_name no)
@@
 			)
 		)
-		(property "Footprint" ""
+		(property "Footprint" "Capacitor_SMD:C_0603_1608Metric_Pad1.08x0.95mm_HandSolder"
 			(at 200.66 73.66 0)
 			(hide yes)
@@
 			(project "flight_controller"
 				(path "/6af40c3f-be19-463b-a9b6-2f3cba853d02/0704ef58-62bc-45a1-abb2-7b7b5f193951"
-					(reference "C1")
+					(reference "C26")
 					(unit 1)
 				)
@@
 			)
 		)
-		(property "Footprint" ""
+		(property "Footprint" "Resistor_SMD:R_0603_1608Metric_Pad0.98x0.95mm_HandSolder"
 			(at 213.36 73.66 0)
 			(hide yes)
@@
 		(dnp no)
 		(fields_autoplaced yes)
-		(property "Reference" "#PWR05"
+		(property "Reference" "#PWR018"
 			(at 82.55 104.14 0)
 			(hide yes)
@@
 			(project "flight_controller"
 				(path "/6af40c3f-be19-463b-a9b6-2f3cba853d02/0704ef58-62bc-45a1-abb2-7b7b5f193951"
-					(reference "#PWR05")
+					(reference "#PWR018")
 					(unit 1)
 				)
@@
 		(dnp no)
 		(fields_autoplaced yes)
-		(property "Reference" "#PWR02"
+		(property "Reference" "#PWR024"
 			(at 229.87 125.73 0)
 			(hide yes)
@@
 			(project "flight_controller"
 				(path "/6af40c3f-be19-463b-a9b6-2f3cba853d02/0704ef58-62bc-45a1-abb2-7b7b5f193951"
-					(reference "#PWR02")
+					(reference "#PWR024")
 					(unit 1)
 				)
@@
 		(dnp no)
 		(fields_autoplaced yes)
-		(property "Reference" "#PWR07"
+		(property "Reference" "#PWR017"
 			(at 63.5 88.9 0)
 			(hide yes)
@@
 			(project "flight_controller"
 				(path "/6af40c3f-be19-463b-a9b6-2f3cba853d02/0704ef58-62bc-45a1-abb2-7b7b5f193951"
-					(reference "#PWR07")
+					(reference "#PWR017")
 					(unit 1)
 				)
@@
 		(dnp no)
 		(fields_autoplaced yes)
-		(property "Reference" "C5"
+		(property "Reference" "C25"
 			(at 137.16 161.2962 0)
 			(show_name no)
@@
 			)
 		)
-		(property "Footprint" ""
+		(property "Footprint" "Capacitor_SMD:C_0603_1608Metric_Pad1.08x0.95mm_HandSolder"
 			(at 134.62 162.56 0)
 			(hide yes)
@@
 			(project "flight_controller"
 				(path "/6af40c3f-be19-463b-a9b6-2f3cba853d02/0704ef58-62bc-45a1-abb2-7b7b5f193951"
-					(reference "C5")
+					(reference "C25")
 					(unit 1)
 				)
@@
 		(dnp no)
 		(fields_autoplaced yes)
-		(property "Reference" "C2"
+		(property "Reference" "C27"
 			(at 247.65 72.3962 0)
 			(show_name no)
@@
 			)
 		)
-		(property "Footprint" ""
+		(property "Footprint" "Capacitor_SMD:C_0603_1608Metric_Pad1.08x0.95mm_HandSolder"
 			(at 245.11 73.66 0)
 			(hide yes)
@@
 			(project "flight_controller"
 				(path "/6af40c3f-be19-463b-a9b6-2f3cba853d02/0704ef58-62bc-45a1-abb2-7b7b5f193951"
-					(reference "C2")
-					(unit 1)
-				)
+					(reference "C27")
+					(unit 1)
+				)
